File: hardware/KiCad/Pocket-Lab-Bench-Power/Pocket-Lab-Bench-Power.kicad_pcb (KiCad board)
At the start: 4 copper layers, 98 x 28 mm, 154 parts, among them J2 Conn_01x04_Pin, J3 Conn_01x04_Pin, J4 Conn_01x02, J5 Conn_01x04_Pin, J6 Conn_01x03_Pin, Q1 CSD87501L, SW1 PS-5850A-6PL, U1 TVS2200DRV, U10 ATtiny3216-S, U11 DC-S011A-D025-20A, U12 TPS259474ARPWR, U15 SY8253ADC, U2 TPS25730SRSMR, U3 BQ25792RQMR, U4 INA226, U5 SY8253ADC, U6 TPS55289RYQR, U7 INA226, U8 ESD122DMYR, U9 TPS70933DBVR

Commit message: PCB routing #1
Parts:
- removed C59, C61: 0.1uF, Capacitor_SMD:C_0603_1608Metric
- removed J3, J5: Conn_01x04_Pin, Connector_PinHeader_2.54mm:PinHeader_1x04_P2.54mm_Vertical
- removed J6: Conn_01x03_Pin, Connector_PinHeader_2.54mm:PinHeader_1x03_P2.54mm_Vertical
- removed R39, R40: 4.7K, Resistor_SMD:R_0603_1608Metric
- removed U10: ATtiny3216-S, Package_SO:SOIC-20W_7.5x12.8mm_P1.27mm
- added C63: 100n, Capacitor_SMD:C_0402_1005Metric, B.Cu at (63.8, 18.2)
- added C64: 10n, Capacitor_SMD:C_0402_1005Metric, B.Cu at (68.6, 15.4)
- added C65: 1u, Capacitor_SMD:C_0402_1005Metric, B.Cu at (69.2, 14.3)
- added C66: 1u, Capacitor_SMD:C_0402_1005Metric, B.Cu at (65.5, 16.8)
- added C67: 100n, Capacitor_SMD:C_0402_1005Metric, B.Cu at (63.8, 25.7)
- added FB1: FerriteBead, Inductor_SMD:L_0603_1608Metric, B.Cu at (65.9, 14.9)
- added R38: 4.7K/1%, Resistor_SMD:R_0603_1608Metric, B.Cu at (62.0, 15.2)
- added R41: 4.7K/1%, Resistor_SMD:R_0603_1608Metric, B.Cu at (61.7, 16.9)
- added U13: STM32L031G6Ux, Package_DFN_QFN:QFN-28_4x4mm_P0.5mm, B.Cu at (64.0, 22.4)
- C52: value 100nF -> 10u; footprint Capacitor_SMD:C_0402_1005Metric -> Capacitor_SMD:C_0603_1608Metric
- C53: value 1uF -> 100n
- R1, R11, R4: footprint Resistor_SMD:R_0603_1608Metric -> Resistor_SMD:R_0402_1005Metric
- R8: value 100 -> 10K; footprint Resistor_SMD:R_0603_1608Metric -> Resistor_SMD:R_0402_1005Metric
- moved C53 10.1 mm to (67.5, 25.2), turned to 0 degrees
- moved C52 7.65 mm to (67.3, 27.5), turned to 0 degrees
- turned R37 to 180 degrees
Connections:
- J2 pad 1: +5V -> GND
- J2 pad 3: Disp_Rst -> SCL
- J2 pad 4: GND -> SDA
- R1 pad 1: 3V3Low -> Encoder_A
- R1 pad 2: Encoder_A -> 3V3Low
- R11 pad 1: Enc_Switch -> GND
- R11 pad 2: GND -> Enc_Switch
- R13 pad 1: 3V3Low -> Alert1
- R13 pad 2: Alert1 -> 3V3Low
- R37 pad 1: SW_State -> 3V3Low
- R37 pad 2: 3V3Low -> SW_State
- R4 pad 1: 3V3Low -> Encoder_B
- R4 pad 2: Encoder_B -> 3V3Low
- R8 pad 2: Net-(J6-Pin_3) -> GND
Routing:
- net (no net): track 0.00 -> 74.2 mm
- net SCL: track 75.4 -> 126.9 mm, vias 4 -> 5
- net Disp_Rst: track 42.5 -> 0.00 mm
- net Disp_En: track 34.9 -> 0.00 mm
- net Disp_Data: track 18.2 -> 0.00 mm
- net Disp_Select: track 18.1 -> 0.00 mm
- net Disp_Clock: track 18.0 -> 0.00 mm
- net PWR_SW: track 51.2 -> 40.3 mm
- net 3V3Low: track 161.3 -> 155.4 mm
- net GND: track 159.5 -> 164.2 mm
- net SW_State: track 39.8 -> 36.2 mm
- net SDA: track 82.8 -> 85.7 mm, vias 6 -> 7
- net Net-(J6-Pin_3): track 2.56 -> 0.00 mm
- net Encoder_A: track 49.1 -> 50.6 mm, vias 0 -> 1
- net Net-(U13-BOOT0): track 12.4 -> 10.8 mm

Commit message: All routing done
Parts:
- added G***: LOGO, LOGO, F.Cu at (41.6, 18.6)
- added J1: Conn_01x05_Pin, Connector_PinHeader_2.54mm:PinHeader_1x05_P2.54mm_Vertical, F.Cu at (62.1, 16.6)
- C60: footprint Capacitor_SMD:C_0805_2012Metric -> Capacitor_SMD:C_1206_3216Metric
- J4: footprint Connector_JST:JST_XH_B2B-XH-A_1x02_P2.50mm_Vertical -> Connector_JST:JST_PH_B2B-PH-K_1x02_P2.00mm_Vertical
- R8: moved to B.Cu
- moved J2 48.7 mm to (86.6, 15.7)
- moved C65 14.6 mm to (61.8, 26.9), turned to 90 degrees
- moved C66 13.8 mm to (60.3, 29.5)
- moved FB1 13.6 mm to (60.4, 27.3), turned to -90 degrees
- moved C64 12.7 mm to (63.2, 26.9), turned to -90 degrees
- moved R38 11.1 mm to (71.3, 21.3), turned to -90 degrees
- moved R8 8.80 mm to (67.9, 24.0), turned to 0 degrees
- moved R41 8.57 mm to (68.8, 21.7), turned to -90 degrees
- moved C67 1.33 mm to (64.4, 26.9), turned to -90 degrees
- moved C63 1.05 mm to (63.8, 19.3)
- moved R37 1.00 mm to (62.0, 19.3), turned to -90 degrees
- moved C60 0.65 mm to (104.5, 32.2)
- moved U13 0.62 mm to (64.0, 23.1)
- moved R11 0.27 mm to (21.4, 36.0), turned to 0 degrees
- moved C53 0.19 mm to (67.7, 25.2)
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Connections:
- U13 pad 21: Net-(J1-Pin_2) -> /SWDIO
- U13 pad 22: Net-(J1-Pin_1) -> /SWCLK
Routing:
- net (no net): track 74.2 -> 0.00 mm
- net +3V3: track 102.2 -> 62.9 mm
- net SCL: track 126.9 -> 93.9 mm, vias 5 -> 7
- net 3V3Low: track 155.4 -> 176.8 mm
- net PWR_SW: track 40.3 -> 58.4 mm
- net /NRST: track 0.00 -> 14.0 mm, vias 0 -> 1
- net /SWCLK: track 0.00 -> 10.6 mm
- net Net-(U13-BOOT0): track 10.8 -> 1.48 mm, vias 1 -> 0
- net SDA: track 85.7 -> 91.2 mm, vias 7 -> 6
- net GND: track 164.2 -> 158.8 mm, vias 65 -> 66
- net /SWDIO: track 0.00 -> 5.17 mm
- net Net-(U13-VDDA): track 0.00 -> 4.38 mm
- net Encoder_A: track 50.6 -> 47.4 mm, vias 1 -> 2
- net +5V: track 69.5 -> 67.0 mm, vias 1 -> 2
- net Net-(C66-Pad2): track 0.00 -> 1.57 mm
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Other:
- board text added: "BenMakesEverything design"
- board text added: "DIO"
- board text added: "NRST"
- board text added: "Rev.0 261207"
- board text added: "STM32 design"
- board text added: "STM32L031"
- board text added: "SWCLK"
- board text removed: "ATTiny3216"
- board text removed: "UPDI"

Commit message: EdgeConnect for programming STM32
Parts:
- added J3: Conn_01x06_Pin, EdgeConnect:Edge_Connect_6, F.Cu at (69.2, 13.0)
Routing:
- net /SWDIO: track 5.17 -> 13.9 mm
- net 3V3Low: track 176.8 -> 181.5 mm
- net /NRST: track 14.0 -> 18.0 mm
- net /SWCLK: track 10.6 -> 14.4 mm
- net +5V: track 67.0 -> 66.3 mm
