File: hardware/KiCad/Pocket-Lab-Bench-Power/Pocket-Lab-Bench-Power.kicad_sch (KiCad schematic)
At the start: 157 parts, among them J1 Conn_01x05_Pin, J2 Conn_01x04_Pin, J3 Conn_01x04_Pin, J4 Conn_01x02, Q1 CSD87501L, SW1 PS-5850A-6PL, U1 TVS2200DRV, U11 DC-S011A-D025-20A, U12 TPS259474ARPWR, U13 STM32L031G6Ux, U15 SY8253ADC, U2 TPS25730SRSMR, U3 BQ25792RQMR, U4 INA226, U5 SY8253ADC, U6 TPS55289RYQR, U7 INA226, U8 ESD122DMYR, U9 TPS70933DBVR

Commit message: PCB routing #1
Parts:
- removed J3: Conn_01x04_Pin, Connector_PinHeader_2.54mm:PinHeader_1x04_P2.54mm_Vertical, symbol Connector:Conn_01x04_Pin
- removed R39, R40: 4.7K, Resistor_SMD:R_0603_1608Metric, symbol Device:R
- added R38, R41: 4.7K/1%, Resistor_SMD:R_0603_1608Metric, symbol Device:R
- C52: value 100n -> 10u; footprint Capacitor_SMD:C_0201_0603Metric -> Capacitor_SMD:C_0603_1608Metric; LCSC C7393837 -> C19702
- C53, C63, C67: footprint Capacitor_SMD:C_0201_0603Metric -> Capacitor_SMD:C_0402_1005Metric; LCSC C7393837 -> C1525
Connections:
- net +3V3: now also J2.2 (Pin_2); no longer J2.3 (Pin_3)
- net 3V3Low: now also R38.2, R41.1
- net Enc_Switch: now also U13.13 (PA7); no longer U13.15 (PB1)
- net GND: now also J2.1 (Pin_1); no longer J2.4 (Pin_4)
- net SCL: now also J2.3 (Pin_3), R41.2; no longer J2.2 (Pin_2)
- net SDA: now also J2.4 (Pin_4), R38.1; no longer J2.1 (Pin_1)
- net SW_State: now also U13.15 (PB1); no longer U13.13 (PA7)
Other:
- note removed: "I2C Header"
- moved on the sheet: J2, R37

Commit message: All routing done
Parts:
- C60: footprint Capacitor_SMD:C_0805_2012Metric -> Capacitor_SMD:C_1206_3216Metric; LCSC (none) -> C412252
- J1: footprint (none) -> Connector_PinHeader_2.54mm:PinHeader_1x05_P2.54mm_Vertical
- J4: footprint Connector_JST:JST_XH_B2B-XH-A_1x02_P2.50mm_Vertical -> Connector_JST:JST_PH_B2B-PH-K_1x02_P2.00mm_Vertical
- U13: LCSC (none) -> C96514
Connections:
- net SWDIO: now reaches J1.2 (Pin_2), U13.21 (PA13)
- net SWCLK: now reaches J1.1 (Pin_1), U13.22 (PA14)
Other:
- moved on the sheet: U8
Changed lines of the file:
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@@
 	)
 	(junction
-		(at 241.3 71.12)
+		(at 104.775 67.31)
 		(diameter 0)
 		(color 0 0 0 0)
 	)
 	(junction
-		(at 86.36 191.77)
+		(at 241.3 71.12)
 		(diameter 0)
 		(color 0 0 0 0)
 	)
 	(junction
-		(at 490.22 233.68)
+		(at 86.36 191.77)
 		(diameter 0)
 		(color 0 0 0 0)
 	)
 	(junction
-		(at 93.98 69.85)
+		(at 490.22 233.68)
 		(diameter 0)
 		(color 0 0 0 0)
@@
 	)
 	(junction
+		(at 94.615 69.85)
+		(diameter 0)
+		(color 0 0 0 0)
+	)
+	(junction
 		(at 535.94 176.53)
 		(diameter 0)
@@
 	)
 	(junction
-		(at 104.14 67.31)
-		(diameter 0)
-		(color 0 0 0 0)
-	)
-	(junction
 		(at 68.58 87.63)
 		(diameter 0)
@@
 	(wire
 		(pts
-			(xy 104.14 67.31) (xy 106.68 67.31)
-		)
-		(stroke
-			(width 0)
-			(type default)
-		)
-	)
-	(wire
-		(pts
 			(xy 252.73 71.12) (xy 264.16 71.12)
 		)
@@
 	(wire
 		(pts
-			(xy 93.98 69.85) (xy 93.98 72.39)
-		)
-		(stroke
-			(width 0)
-			(type default)
-		)
-	)
-	(wire
-		(pts
 			(xy 448.31 60.96) (xy 448.31 58.42)
 		)
@@
 	(wire
 		(pts
+			(xy 94.615 69.85) (xy 94.615 78.74)
+		)
+		(stroke
+			(width 0)
+			(type default)
+		)
+	)
+	(wire
+		(pts
 			(xy 97.79 295.91) (xy 101.6 295.91)
 		)
@@
 		)
 	)
+	(wire
+		(pts
+			(xy 104.775 67.31) (xy 104.775 78.74)
+		)
+		(stroke
+			(width 0)
+			(type default)
+		)
+	)
 	(polyline
 		(pts
@@
 	(wire
 		(pts
-			(xy 104.14 67.31) (xy 104.14 72.39)
-		)
-		(stroke
-			(width 0)
-			(type default)
-		)
-	)
-	(wire
-		(pts
 			(xy 125.73 76.2) (xy 127 76.2)
 		)
@@
 	(wire
 		(pts
-			(xy 93.98 69.85) (xy 106.68 69.85)
-		)
-		(stroke
-			(width 0)
-			(type default)
-		)
-	)
-	(wire
-		(pts
 			(xy 200.66 30.48) (xy 200.66 33.02)
 		)
@@
 	(wire
 		(pts
+			(xy 99.695 109.22) (xy 99.695 111.76)
+		)
+		(stroke
+			(width 0)
+			(type default)
+		)
+	)
+	(wire
+		(pts
 			(xy 320.04 186.69) (xy 320.04 191.77)
 		)
@@
 	(wire
 		(pts
+			(xy 94.615 69.85) (xy 106.68 69.85)
+		)
+		(stroke
+			(width 0)
+			(type default)
+		)
+	)
+	(wire
+		(pts
 			(xy 228.6 175.26) (xy 228.6 179.07)
 		)
@@
 	(wire
 		(pts
-			(xy 66.04 67.31) (xy 104.14 67.31)
-		)
-		(stroke
-			(width 0)
-			(type default)
-		)
-	)
-	(wire
-		(pts
 			(xy 568.96 81.28) (xy 568.96 83.82)
 		)
@@
 	(wire
 		(pts
-			(xy 99.06 102.87) (xy 99.06 105.41)
+			(xy 229.87 91.44) (xy 229.87 78.74)
 		)
 		(stroke
@@
 	(wire
 		(pts
-			(xy 229.87 91.44) (xy 229.87 78.74)
+			(xy 80.01 36.83) (xy 80.01 40.64)
 		)
 		(stroke
@@
 	(wire
 		(pts
-			(xy 80.01 36.83) (xy 80.01 40.64)
+			(xy 436.88 93.98) (xy 436.88 100.33)
 		)
 		(stroke
@@
 	(wire
 		(pts
-			(xy 436.88 93.98) (xy 436.88 100.33)
+			(xy 53.34 172.72) (xy 53.34 170.18)
 		)
 		(stroke
@@
 	(wire
 		(pts
-			(xy 53.34 172.72) (xy 53.34 170.18)
+			(xy 66.04 67.31) (xy 104.775 67.31)
 		)
 		(stroke
@@
 	(wire
 		(pts
+			(xy 104.775 67.31) (xy 106.68 67.31)
+		)
+		(stroke
+			(width 0)
+			(type default)
+		)
+	)
+	(wire
+		(pts
 			(xy 27.94 87.63) (xy 34.29 87.63)
 		)
@@
 	(wire
 		(pts
-			(xy 66.04 69.85) (xy 93.98 69.85)
+			(xy 66.04 69.85) (xy 94.615 69.85)
 		)
 		(stroke
@@
 		)
 	)
+	(label "SWDIO"
+		(at 255.27 267.97 0)
+		(effects
+			(font
+				(size 1.27 1.27)
+			)
+			(justify left bottom)
+		)
+	)
 	(label "NRST"
 		(at 265.43 257.175 0)
@@
 		)
 	)
+	(label "SWCLK"
+		(at 255.27 270.51 0)
+		(effects
+			(font
+				(size 1.27 1.27)
+			)
+			(justify left bottom)
+		)
+	)
 	(label "Charger_D_P"
 		(at 106.68 69.85 0)
@@
 			)
 		)
+		(property "LCSC" "C96514"
+			(at 215.9 252.73 0)
+			(effects
+				(font
+					(size 1.27 1.27)
+				)
+				(hide yes)
+			)
+		)
 		(pin "28"
 		)
@@
 			)
 		)
-		(property "Footprint" "Connector_JST:JST_XH_B2B-XH-A_1x02_P2.50mm_Vertical"
+		(property "Footprint" "Connector_JST:JST_PH_B2B-PH-K_1x02_P2.00mm_Vertical"
 			(at 299.72 163.83 0)
 			(effects
@@
 			)
 		)
-		(property "Footprint" "Capacitor_SMD:C_0805_2012Metric"
+		(property "Footprint" "Capacitor_SMD:C_1206_3216Metric"
 			(at 510.2352 241.3 0)
 			(effects
@@
 			)
 		)
+		(property "LCSC" "C412252"
+			(at 509.27 237.49 0)
+			(effects
+				(font
+					(size 1.27 1.27)
+				)
+				(hide yes)
+			)
+		)
 		(pin "1"
 		)
@@
 	(symbol
 		(lib_id "ESD122DMYR:ESD122DMYR")
-		(at 99.06 87.63 90)
+		(at 99.695 93.98 90)
 		(unit 1)
 		(exclude_from_sim no)
@@
 		(dnp no)
 		(property "Reference" "U8"
-			(at 100.838 100.076 90)
+			(at 101.473 106.426 90)
 			(effects
 				(font
@@
 		)
 		(property "Value" "ESD122DMYR"
-			(at 100.838 103.886 90)
+			(at 101.473 110.236 90)
 			(effects
 				(font
@@
 		)
 		(property "Footprint" "MyParts:DMY0003A"
-			(at 99.06 87.63 0)
+			(at 99.695 93.98 0)
 			(effects
 				(font
@@
 		)
 		(property "Datasheet" "https://www.ti.com/lit/gpn/esd122"
-			(at 99.06 87.63 0)
+			(at 99.695 93.98 0)
 			(effects
 				(font
@@
 		)
 		(property "Description" ""
-			(at 99.06 87.63 0)
+			(at 99.695 93.98 0)
 			(effects
 				(font
@@
 		)
 		(property "LCSC Part" "C1975871"
-			(at 99.06 87.63 90)
+			(at 99.695 93.98 90)
 			(effects
 				(font
@@
 	(symbol
 		(lib_id "power:GND")
-		(at 99.06 105.41 0)
+		(at 99.695 111.76 0)
 		(unit 1)
 		(exclude_from_sim no)
@@
 		(fields_autoplaced yes)
 		(property "Reference" "#PWR029"
-			(at 99.06 111.76 0)
+			(at 99.695 118.11 0)
 			(effects
 				(font
@@
 		)
 		(property "Value" "GND"
-			(at 99.06 110.49 0)
+			(at 99.695 116.84 0)
 			(effects
 				(font
@@
 		)
 		(property "Footprint" ""
-			(at 99.06 105.41 0)
+			(at 99.695 111.76 0)
 			(effects
 				(font
@@
 		)
 		(property "Datasheet" ""
-			(at 99.06 105.41 0)
+			(at 99.695 111.76 0)
 			(effects
 				(font
@@
 		)
 		(property "Description" "Power symbol creates a global label with name \"GND\" , ground"
-			(at 99.06 105.41 0)
+			(at 99.695 111.76 0)
 			(effects
 				(font
@@
 			)
 		)
-		(property "Footprint" ""
+		(property "Footprint" "Connector_PinHeader_2.54mm:PinHeader_1x05_P2.54mm_Vertical"
 			(at 279.4 265.43 0)
 			(effects

Commit message: EdgeConnect for programming STM32
Parts:
- added J3: Conn_01x06_Pin, EdgeConnect:Edge_Connect_6, symbol Connector:Conn_01x06_Pin
Connections:
- net 3V3Low: now also J3.1 (Pin_1)
- net GND: now also J3.5 (Pin_5)
- net NRST: now also J3.3 (Pin_3)
- net SWCLK: now also J3.4 (Pin_4)
- net SWDIO: now also J3.2 (Pin_2)
- no-connect marks 23 -> 24
Other:
- note added: "MCU Programming Headers"
- note removed: "MCU Programming Header"
